Commit message: data loop started

File: models/X5.urdf (robot description, URDF)
Before this commit: robot X5, 8 links, 7 joints
Links:
- link link6: mass 0.581000 -> 0.571000

Commit message: chunked sending; needs improvement in future

File: models/X5.urdf (robot description, URDF)
Before this commit: robot X5, 8 links, 7 joints
Links:
- link link6: mass 0.571000 -> 0.651000
